File: STM32F070F6P6.sch (KiCad schematic (older format))
At the start: 9 parts, among them U5 16Mhz, U6 7_Pins_Header_PA0_PA6, U7 STM32F070F6P6, U8 7_Pins_Header_PA7_PA14

Commit message: Updated to Rev2.0
Parts:
- removed U6: 7_Pins_Header_PA0_PA6, Footprints:7_Pins_Headers, symbol 7_Pins_Header_PA0_PA6
- removed U7: STM32F070F6P6, Footprints:TSSOP20, symbol STM32F070F6P6
- removed U8: 7_Pins_Header_PA7_PA14, Footprints:7_Pins_Headers, symbol 7_Pins_Header_PA7_PA14
- added C401: C, Footprints2:SMD_CAP_1210, symbol C
- added JP401: Jumper_NO_Small, conn-test:JUMPER-SOLDER-SMD, symbol Jumper_NO_Small
- added P401, P403: CONN_01X12, Pin_Headers:Pin_Header_Straight_1x12_Pitch2.54mm, symbol CONN_01X12
- added P402: CONN_01X02, rascalmicro-kicad-footprints:s2b-ph-sm4-tb, symbol CONN_01X02
- added U402: STM32F401CEU6, Housings_DFN_QFN:QFN-48-1EP_7x7mm_Pitch0.5mm, symbol STM32F401CEU6
- renumbered FID1 to FID401, FID2 to FID402, R2 to R401, R3 to R402, R4 to R403, U5 to U401
Connections:
- net labels added: PA0, PA1, PA15, PA2, PA3, PA4, PA5, PA6, PA7, PB10, PB12, PB13, PB14, PB15, PB2, PB3, PB4, PB5, PB6, PB7, PB8, PB9
- wire segments 44 -> 80
- no-connect marks 0 -> 7
Other:
- note added: "BOOT0, SWCLK, SWDIO, USB+, USB-, NRST, VBUS,"
- moved on the sheet: R401, U401
