File: AMW007R.sch (KiCad schematic (older format))
At the start: 8 parts, among them U1 AMW007R, U2 2.4Ghz_Ant1

Commit message: Updated..
Parts:
- U1: footprint Footprints2:AMW007R -> (none)
Changed lines of the file:
@@
 LIBS:tactile_button
 LIBS:NEOM_0
+LIBS:amw007r
 LIBS:NEOM_0-cache
 EELAYER 25 0
@@
 $EndComp
 $Comp
-L GND #PWR023
+L GND #PWR1
 U 1 1 5A360869
 P 1550 2500
-F 0 "#PWR023" H 1550 2250 50  0001 C CNN
+F 0 "#PWR1" H 1550 2250 50  0001 C CNN
 F 1 "GND" H 1550 2350 50  0000 C CNN
 F 2 "" H 1550 2500 50  0000 C CNN
@@
 $EndComp
 $Comp
-L GND #PWR024
+L GND #PWR4
 U 1 1 5A36088B
 P 6650 5300
-F 0 "#PWR024" H 6650 5050 50  0001 C CNN
+F 0 "#PWR4" H 6650 5050 50  0001 C CNN
 F 1 "GND" H 6650 5150 50  0000 C CNN
 F 2 "" H 6650 5300 50  0000 C CNN
@@
 $EndComp
 $Comp
-L GND #PWR025
+L GND #PWR5
 U 1 1 5A3608AD
 P 7400 3900
-F 0 "#PWR025" H 7400 3650 50  0001 C CNN
+F 0 "#PWR5" H 7400 3650 50  0001 C CNN
 F 1 "GND" H 7400 3750 50  0000 C CNN
 F 2 "" H 7400 3900 50  0000 C CNN
@@
 $EndComp
 $Comp
-L GND #PWR026
+L GND #PWR6
 U 1 1 5A3608CF
 P 8200 3900
-F 0 "#PWR026" H 8200 3650 50  0001 C CNN
+F 0 "#PWR6" H 8200 3650 50  0001 C CNN
 F 1 "GND" H 8200 3750 50  0000 C CNN
 F 2 "" H 8200 3900 50  0000 C CNN
@@
 $EndComp
 $Comp
-L GND #PWR027
+L GND #PWR7
 U 1 1 5A3608F1
 P 9550 2850
-F 0 "#PWR027" H 9550 2600 50  0001 C CNN
+F 0 "#PWR7" H 9550 2600 50  0001 C CNN
 F 1 "GND" H 9550 2700 50  0000 C CNN
 F 2 "" H 9550 2850 50  0000 C CNN
@@
 Connection ~ 8200 3350
 $Comp
-L +3.3V #PWR028
+L +3.3V #PWR3
 U 1 1 5A360EC1
 P 6500 1650
-F 0 "#PWR028" H 6500 1500 50  0001 C CNN
+F 0 "#PWR3" H 6500 1500 50  0001 C CNN
 F 1 "+3.3V" H 6500 1790 50  0000 C CNN
 F 2 "" H 6500 1650 50  0000 C CNN
@@
 $EndComp
 $Comp
-L +3.3V #PWR029
+L +3.3V #PWR2
 U 1 1 5A360EEB
 P 1550 5050
-F 0 "#PWR029" H 1550 4900 50  0001 C CNN
+F 0 "#PWR2" H 1550 4900 50  0001 C CNN
 F 1 "+3.3V" H 1550 5190 50  0000 C CNN
 F 2 "" H 1550 5050 50  0000 C CNN
@@
 $Comp
 L AMW007R~ U1
-U 1 1 5A367F40
+U 1 1 5A420784
 P 4600 3500
 F 0 "U1" H 3000 1550 60  0000 C CNN
 F 1 "AMW007R" H 3150 5550 60  0000 C CNN
-F 2 "Footprints2:AMW007R" H 3000 4650 60  0001 C CNN
-F 3 "" H 3000 4650 60  0001 C CNN
+F 2 "" H 3000 4650 60  0000 C CNN
+F 3 "" H 3000 4650 60  0000 C CNN
 	1    4600 3500
 	1    0    0    -1
