File: NEOM_0.kicad_pcb (KiCad board)
At the start: 4 copper layers, 27 x 50.3 mm, 31 parts, among them P1 CONN_01X09, P402 CONN_01X02, P403 CONN_01X12, SW201 SPST, U1 AMW007Rr, U2 2.4Ghz_Ant1, U201 LM3940, U3 USBLC6-2, U302 USB_Micro_B, U401 16Mhz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

Commit message: Updated...
Parts:
- added REF***: OSHW-Logo2_7.3x6mm_Copper, Symbols:OSHW-Logo2_7.3x6mm_SilkScreen, B.Cu at (33.5, 34.7)
- moved FID401 21.8 mm to (22.2, 67.2)
